File: $RC_StellarisBoard.sch (KiCad schematic (older format))
At the start: 46 parts, among them K1 CONN_3, K2 CONN_3, K3 CONN_3, K4 CONN_3, K5 CONN_3, P1 CONN_2, P2 CONN_1, P3 CONN_1, P4 CONN_1, P5 CONN_1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

Commit message: versao 1 placa
Parts:
- removed Q1: MOSFET_P, ~, symbol MOSFET_P
- added Q1: MOS_P_123, ~, symbol MOS_P_123
Changed lines of the file:
@@
 LIBS:amc6821
 LIBS:TPS62112
+LIBS:mos_p_(1-2-3)
 LIBS:RC_StellarisBoard-cache
 EELAYER 27 0
@@
 $EndComp
 $Comp
-L MOSFET_P Q1
-U 1 1 52C8A420
-P 2650 2700
-F 0 "Q1" H 2650 2890 60  0000 R CNN
-F 1 "MOSFET_P" V 2650 2520 60  0000 R CNN
-F 2 "~" H 2650 2700 60  0000 C CNN
-F 3 "~" H 2650 2700 60  0000 C CNN
-	1    2650 2700
-	0    1    -1   0
-$EndComp
-$Comp
 L CONN_2 P6
 U 1 1 52C97D7A
@@
 Connection ~ 2200 5750
 Connection ~ 2200 5550
+$Comp
+L MOS_P_123 Q1
+U 1 1 52C9AD33
+P 2650 2700
+F 0 "Q1" H 2650 2890 60  0000 R CNN
+F 1 "MOS_P_123" H 2650 2520 60  0000 R CNN
+F 2 "~" H 2650 2700 60  0000 C CNN
+F 3 "~" H 2650 2700 60  0000 C CNN
+	1    2650 2700
+	0    1    -1   0
+$EndComp
 $EndSCHEMATC
