File: $RC_StellarisBoard.sch (KiCad schematic (older format))
At the start: 68 parts, among them K1 CONN_3, K2 CONN_3, K3 CONN_3, K4 CONN_3, K5 CONN_3, P1 CONN_2, P10 XT-60 out, P11 CONN_1, P2 CONN_1, P3 CONN_1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

Commit message: versao com tudo
Parts:
- gave numbers to parts that had none: 7
