File: buck-boost.kicad_pcb (KiCad board)
At the start: 2 copper layers, 14.5 x 17.8 mm, 6 parts, among them P1 CONN_2, P2 CONN_2, U2 LM3668_DQB_12_SDF12A

Commit message: feito
Parts:
- added C3: CP1, SM1206POL, F.Cu at (226.4, 126.1)
- added C4: C, SM1206, F.Cu at (222.9, 126.1)
- added C5: C, SM1206, F.Cu at (229.9, 120.3)
- added C6: CP1, SM2512, F.Cu at (224.9, 118.7)
- added L2: INDUCTOR, bournes_7.8, F.Cu at (236.3, 120.1)
- added P3: CONN_2, SparkFun-1X02_LOCK, F.Cu at (218.9, 128.4)
- added P4: CONN_2, SparkFun-1X02_LOCK, F.Cu at (219.2, 117.5)
- added R1: R, SM0603, F.Cu at (228.1, 131.4)
- added U1: TPS6211_QFN16-4X4, QFN65P400X400X100-17N, F.Cu at (231.5, 128.1)
Connections:
- net +BATT renamed +5V
Routing:
- net GND: track 49.2 -> 155.1 mm
- net +5V: track 41.1 -> 84.6 mm
- net +BATT: track 0.00 -> 32.1 mm
- net N-000002: track 0.00 -> 14.8 mm
