File: buck-boost.sch (KiCad schematic (older format))
At the start: 6 parts, among them P1 CONN_2, P2 CONN_2, U2 LM3668_DQB_12_SDF12A

Commit message: feito
Parts:
- added C3, C6: CP1, symbol CP1
- added C4, C5: C, symbol C
- added L2: INDUCTOR, symbol INDUCTOR
- added P3, P4: CONN_2, symbol CONN_2
- added R1: R, symbol R
- added U1: TPS6211_QFN16-4X4, QFN16, symbol TPS6211_QFN16-4X4
Connections:
- net +BATT: now also C3.1, C4.1, P3.1 (P1), R1.1, R1.2, U1.2 (VIN), U1.3 (VIN), U1.4 (EN), U1.8 (VINA); no longer C2.1, P2.1 (P1), U2.11 (VSEL), U2.5 (PVIN), U2.6 (EN), U2.7 (VDD)
- net GND: now also C3.2, C4.2, C5.2, C6.2, P3.2 (PM), P4.2 (PM), U1.1 (PGND), U1.11 (GND), U1.12 (GND), U1.13 (PG), U1.16 (PGND), U1.17 (PWPD), U1.5 (SYNC), U1.6 (LBO), U1.7 (LBI), U1.9 (AGND)
- new net: L2.1, U1.14 (SW), U1.15 (SW)
- new net +5V: C2.1, C5.1, C6.1, L2.2, P2.1 (P1), P4.1 (P1), U1.10 (FB), U2.11 (VSEL), U2.5 (PVIN), U2.6 (EN), U2.7 (VDD)
